File: KiCAD/aux/aux.kicad_pcb (KiCad board)
At the start: 2 copper layers, 140 x 127.5 mm, 169 parts, among them J1 PMOD_male_2row, J2 Conn_01x12_Socket, J3 Conn_Coaxial_Small, J4 Conn_Coaxial_Small, J5 Conn_Coaxial_Small, J6 Conn_Coaxial_Small, J7 Conn_Coaxial_Small, J8 1803426, J9 1758018, Q1 SQJ746ELP-T1_GE3, T1 WB1-1L, T2 WB1-1L, T3 WB1-1L, T4 WB1-1L, T5 LM-NP-1001-B1L, U1 AD8055ARTZ-R2, U10 TPS563201, U11 LDL1117S50R_, U12 LT3045xMSE, U13 LM5161PWP, U14 LM5161PWP, U2 AD8055ARTZ-R2, U3 AD8055ARTZ-R2, U4 AD8055ARTZ-R2, U5 AD8055ARTZ-R2, U6 OPA171AIDBVR, U7 DAC121S101CIMKX_NOPB, U8 AP74502QTA8-7, U9 MIC29302WU

Commit message: Reworked, now with IRIG option board complete
Parts:
- removed the C28 at (96.5, 128.0)
- removed the C30 at (119.0, 126.4)
- removed the C31 at (137.2, 130.8)
- removed the C32 at (134.4, 130.8)
- removed the C33 at (108.8, 137.4)
- removed the C34 at (152.6, 133.2)
- removed the C35 at (136.2, 146.0)
- removed the C36 at (161.8, 136.2)
- removed the C37 at (159.2, 136.2)
- removed the C38 at (115.2, 142.8)
- removed the C39 at (112.0, 142.8)
- removed the C40 at (168.8, 74.6)
- removed the C41 at (152.8, 80.4)
- removed the C42 at (149.2, 80.4)
- removed the C43 at (149.4, 89.2)
- removed the C44 at (185.0, 83.2)
- removed the C45 at (150.0, 94.0)
- removed the C49 at (182.2, 61.4)
- removed the C51 at (185.0, 86.4)
- removed J2: Conn_01x12_Socket, Connector_PinSocket_2.54mm:PinSocket_1x12_P2.54mm_Vertical
- removed the L5 at (146.1, 151.6)
- removed L7: DRQ127-100-R, ! Eaton:DRQ127
- removed the R25 at (116.4, 126.4)
- removed the R26 at (116.6, 131.6)
- removed the R27 at (114.0, 131.6)
- removed the R28 at (156.8, 148.0)
- removed the R29 at (91.4, 142.4)
- removed the R30 at (156.8, 142.4)
- removed the R34 at (168.7, 84.0)
- removed the R35 at (158.2, 94.2)
- removed the R36 at (148.4, 94.0)
- removed the R37 at (172.1, 83.2)
- removed the R38 at (185.0, 88.0)
- removed the R40 at (169.7, 86.6)
- removed the R41 at (185.0, 89.6)
- removed the R43 at (168.6, 114.2)
- removed ST1: ~, ! Scott:star5tie
- removed the U10 at (155.9, 134.6)
- removed the U12 at (144.1, 92.4)
- removed the U13 at (177.7, 83.0)
- removed the U8 at (160.4, 74.2)
- removed the U9 at (126.4, 135.7)
- added C10: 10uf, Capacitor_SMD:C_1206_3216Metric_Pad1.33x1.80mm_HandSolder, F.Cu at (150.0, 69.8)
- added C11: 100uf polymer, Capacitor_THT:CP_Radial_D5.0mm_P2.00mm, F.Cu at (144.0, 65.3)
- added C12: 22uf, Capacitor_SMD:C_1206_3216Metric_Pad1.33x1.80mm_HandSolder, F.Cu at (155.8, 138.0)
- added C13: 1uf, Capacitor_SMD:C_1206_3216Metric_Pad1.33x1.80mm_HandSolder, F.Cu at (171.2, 134.5)
- added C14: 82pf, Capacitor_SMD:C_0402_1005Metric_Pad0.74x0.62mm_HandSolder, F.Cu at (167.0, 142.8)
- added C15: 5.1pf, Capacitor_SMD:C_0402_1005Metric_Pad0.74x0.62mm_HandSolder, F.Cu at (164.8, 141.8)
- added C16: 39uf, Capacitor_SMD:C_1206_3216Metric_Pad1.33x1.80mm_HandSolder, F.Cu at (168.0, 114.2)
- added C17: 39uf, Capacitor_SMD:C_1206_3216Metric_Pad1.33x1.80mm_HandSolder, F.Cu at (168.0, 116.8)
- added C20: 10uf, Capacitor_SMD:C_1206_3216Metric_Pad1.33x1.80mm_HandSolder, F.Cu at (149.5, 74.5)
- added C21: 100uf polymer, Capacitor_THT:CP_Radial_D5.0mm_P2.00mm, F.Cu at (144.0, 71.8)
- added C22: 33nf, Capacitor_SMD:C_0402_1005Metric_Pad0.74x0.62mm_HandSolder, F.Cu at (162.8, 142.2)
- added C23: 150pf, Capacitor_SMD:C_0402_1005Metric_Pad0.74x0.62mm_HandSolder, F.Cu at (161.8, 142.2)
- added C24: 10uf, Capacitor_SMD:C_1206_3216Metric_Pad1.33x1.80mm_HandSolder, F.Cu at (149.5, 79.2)
- added C25: 100uf polymer, Capacitor_THT:CP_Radial_D5.0mm_P2.00mm, F.Cu at (144.0, 78.3)
- added C3: 10uf, Capacitor_SMD:C_1206_3216Metric_Pad1.33x1.80mm_HandSolder, F.Cu at (182.0, 66.8)
- added C4: 10uf, Capacitor_SMD:C_1206_3216Metric_Pad1.33x1.80mm_HandSolder, F.Cu at (190.0, 74.4)
- added C5: 220nf, Capacitor_SMD:C_1206_3216Metric_Pad1.33x1.80mm_HandSolder, F.Cu at (185.6, 82.6)
- added C6: 0.1uf, Capacitor_SMD:C_1206_3216Metric_Pad1.33x1.80mm_HandSolder, F.Cu at (181.8, 81.4)
- added C64: 0.1uf, Capacitor_SMD:C_1206_3216Metric_Pad1.33x1.80mm_HandSolder, F.Cu at (167.3, -68.8)
- added C68: 10uf, Capacitor_SMD:C_1206_3216Metric_Pad1.33x1.80mm_HandSolder, F.Cu at (117.4, 148.6)
- added C69: 10uf, Capacitor_SMD:C_1206_3216Metric_Pad1.33x1.80mm_HandSolder, F.Cu at (117.4, 151.8)
- added C8: 100nf, Capacitor_SMD:C_0603_1608Metric_Pad1.08x0.95mm_HandSolder, F.Cu at (158.0, 131.8)
- added D10: LED, LED_SMD:LED_0805_2012Metric_Pad1.15x1.40mm_HandSolder, F.Cu at (107.8, -30.6)
- added D11: LED, LED_SMD:LED_0805_2012Metric_Pad1.15x1.40mm_HandSolder, F.Cu at (107.8, -27.6)
- added D12: LED, LED_SMD:LED_0805_2012Metric_Pad1.15x1.40mm_HandSolder, F.Cu at (108.8, 145.2)
- added F2: RUEF250, ! Littlefuse:FUS_RUEF250_TYCO_TYC, F.Cu at (190.6, 87.4)
- added FB4: BLM31PG601, Inductor_SMD:L_1206_3216Metric_Pad1.22x1.90mm_HandSolder, F.Cu at (121.8, 150.2)
- added H3: MountingHole, MountingHole:MountingHole_3.2mm_M3, F.Cu at (64.0, 39.0)
- added H4: MountingHole, MountingHole:MountingHole_3.2mm_M3, F.Cu at (201.0, 39.0)
- added H5: MountingHole, MountingHole:MountingHole_3.2mm_M3, F.Cu at (64.0, 150.0)
- added H6: MountingHole, MountingHole:MountingHole_3.2mm_M3, F.Cu at (201.0, 150.0)
- added H7: MountingHole_Pad, MountingHole:MountingHole_2.7mm_M2.5_Pad, F.Cu at (52.0, 46.0)
- added H8: MountingHole_Pad, MountingHole:MountingHole_2.7mm_M2.5_Pad, F.Cu at (52.0, 104.0)
- added J13: Conn_01x12_Socket, Connector_PinSocket_2.54mm:PinSocket_1x12_P2.54mm_Vertical, F.Cu at (81.7, 131.0)
- added J17: Conn_02x20_Odd_Even, Connector_PinHeader_2.54mm:PinHeader_2x20_P2.54mm_Vertical, F.Cu at (50.5, 50.9)
- added J3: Conn_01x02_Pin, Connector_PinHeader_2.54mm:PinHeader_1x02_P2.54mm_Vertical, F.Cu at (104.5, 148.4)
- added J7: PJ-037A, ! CUI Devices:CUI_PJ-037A, F.Cu at (193.0, 57.5)
- added L1: HP6-0090L, ! Coilcraft:HP6-0090L, F.Cu at (145.8, 104.0)
- added MOD1: ~, ! Scott:Adafruit Ultimate GPS Breakout v3, F.Cu at (178.9, 124.4)
- added MOD7: Conn_02x04_Odd_Even, ! Scott:RCB-F9T-0, F.Cu at (193.8, 120.4)
- added Q2: SQJ746ELP-T1_GE3, ! Vishay:PowerPAK_SO-8L-2_DUAL_VIS, F.Cu at (179.6, 72.4)
- added Q3: GSFD0650, Package_TO_SOT_SMD:TO-252-2, F.Cu at (155.8, 124.2)
- added Q4: GSFD0650, Package_TO_SOT_SMD:TO-252-2, F.Cu at (163.0, 124.2)
- added Q5: IRLML6344TRPBF, ! Infineon:TRANS_IRLML6344TRPBF, F.Cu at (93.2, 148.4)
- added R1: 1M, Resistor_SMD:R_0402_1005Metric_Pad0.72x0.64mm_HandSolder, F.Cu at (158.8, 145.2)
- added R10: 24.3K, Resistor_SMD:R_1206_3216Metric_Pad1.30x1.75mm_HandSolder, F.Cu at (178.2, 89.0)
- added R11: 36.5K, Resistor_SMD:R_1206_3216Metric_Pad1.30x1.75mm_HandSolder, F.Cu at (175.2, 79.0)
- added R12: 10K, Resistor_SMD:R_1206_3216Metric_Pad1.30x1.75mm_HandSolder, F.Cu at (182.0, 91.0)
- added R13: 10K, Resistor_SMD:R_1206_3216Metric_Pad1.30x1.75mm_HandSolder, F.Cu at (175.2, 84.0)
- added R16: 2.26K, Resistor_SMD:R_0402_1005Metric_Pad0.72x0.64mm_HandSolder, F.Cu at (158.8, 143.2)
- added R17: 25K, Resistor_SMD:R_0402_1005Metric_Pad0.72x0.64mm_HandSolder, F.Cu at (158.8, 144.2)
- added R18: 210K, Resistor_SMD:R_0402_1005Metric_Pad0.72x0.64mm_HandSolder, F.Cu at (164.8, 142.8)
- added R19: 50K, Resistor_SMD:R_0402_1005Metric_Pad0.72x0.64mm_HandSolder, F.Cu at (164.8, 143.8)
- added R2: 15.4K, Resistor_SMD:R_0402_1005Metric_Pad0.72x0.64mm_HandSolder, F.Cu at (158.8, 142.2)
- added R20: 10mohm, Resistor_SMD:R_1206_3216Metric_Pad1.30x1.75mm_HandSolder, F.Cu at (169.5, 129.2)
- added R22: 11.5K, Resistor_SMD:R_0402_1005Metric_Pad0.72x0.64mm_HandSolder, F.Cu at (164.8, 144.8)
- added R4: 75K, Resistor_SMD:R_1206_3216Metric_Pad1.30x1.75mm_HandSolder, F.Cu at (190.0, 97.2)
- added R49: 10K, Resistor_SMD:R_0603_1608Metric_Pad0.98x0.95mm_HandSolder, B.Cu at (147.5, 98.5)
- added R50: 100K, Resistor_SMD:R_1206_3216Metric_Pad1.30x1.75mm_HandSolder, F.Cu at (89.6, 148.6)
- added R51: 560, Resistor_SMD:R_1206_3216Metric_Pad1.30x1.75mm_HandSolder, F.Cu at (103.3, 145.2)
- added R6: 10K, Resistor_SMD:R_1206_3216Metric_Pad1.30x1.75mm_HandSolder, F.Cu at (184.8, 97.2)
- added R7: 10K, Resistor_SMD:R_1206_3216Metric_Pad1.30x1.75mm_HandSolder, F.Cu at (181.1, 102.5)
- added R8: 560, Resistor_SMD:R_1206_3216Metric_Pad1.30x1.75mm_HandSolder, F.Cu at (182.0, 64.4)
- added R9: 3.3K, Resistor_SMD:R_1206_3216Metric_Pad1.30x1.75mm_HandSolder, F.Cu at (187.6, 68.2)
- added REF**: KiCad-Logo2_8mm_SilkScreen, Symbol:KiCad-Logo2_8mm_SilkScreen, F.Cu at (213.2, -17.8)
- added REF**: OSHW-Logo2_24.3x20mm_SilkScreen, Symbol:OSHW-Logo2_24.3x20mm_SilkScreen, F.Cu at (202.1, -76.6)
- added TP10: TestPoint_Probe, TestPoint:TestPoint_Pad_2.0x2.0mm, F.Cu at (143.9, -32.6)
- added TP11: TestPoint_Probe, TestPoint:TestPoint_Pad_2.0x2.0mm, F.Cu at (143.9, -28.5)
- added TP9: TestPoint_Probe, TestPoint:TestPoint_Pad_2.0x2.0mm, F.Cu at (143.9, -36.6)
- added U1: AP74502QTA8-7, ! Diodes Incorporated:SOT65P280X110-8N, F.Cu at (178.0, 99.3)
- added U15: TPS563201, Package_TO_SOT_SMD:SOT-23-6, B.Cu at (154.2, 96.0)
- added U16: MIC29302WU, Package_TO_SOT_SMD:TO-263-5_TabPin3, F.Cu at (112.7, 107.0)
- added U2: AP22654WU-7, ! Diodes Incorporated:SOT95P280X82-6N, F.Cu at (186.1, 72.2)
- added U3: AP74502QTA8-7, ! Diodes Incorporated:SOT65P280X110-8N, F.Cu at (178.7, 80.2)
- added U6: LM25116MHX_NOPB, ! Texas Instruments:SOP65P640X110-21N, F.Cu at (162.0, 137.0)
- C1: value 0.1uf -> 10uf
- C46: value 10uf -> 22uf; footprint Capacitor_SMD:C_0603_1608Metric_Pad1.08x0.95mm_HandSolder -> Capacitor_SMD:C_1206_3216Metric_Pad1.33x1.80mm_HandSolder; moved to B.Cu
- C47: value 0.1uf -> 22uf; footprint Capacitor_SMD:C_0603_1608Metric_Pad1.08x0.95mm_HandSolder -> Capacitor_SMD:C_1206_3216Metric_Pad1.33x1.80mm_HandSolder
- C48, C58: value 3.3nf -> 10uf; footprint Capacitor_SMD:C_0603_1608Metric_Pad1.08x0.95mm_HandSolder -> Capacitor_SMD:C_1206_3216Metric_Pad1.33x1.80mm_HandSolder; moved to B.Cu
- C50: value 10uf -> 0.01uf C0G; footprint Capacitor_SMD:C_0603_1608Metric_Pad1.08x0.95mm_HandSolder -> Capacitor_SMD:C_1206_3216Metric_Pad1.33x1.80mm_HandSolder
- C52: value 27nf -> 22uf; footprint Capacitor_SMD:C_0603_1608Metric_Pad1.08x0.95mm_HandSolder -> Capacitor_SMD:C_1206_3216Metric_Pad1.33x1.80mm_HandSolder
- C53: value 1uf -> 10uf; footprint Capacitor_SMD:C_0603_1608Metric_Pad1.08x0.95mm_HandSolder -> Capacitor_SMD:C_1206_3216Metric_Pad1.33x1.80mm_HandSolder; moved to B.Cu
- C54: value 100uf polymer -> 10uf; footprint Capacitor_THT:CP_Radial_D5.0mm_P2.00mm -> Capacitor_SMD:C_1206_3216Metric_Pad1.33x1.80mm_HandSolder; moved to B.Cu
- C55: value 0.1uf -> 10uf; footprint Capacitor_SMD:C_0603_1608Metric_Pad1.08x0.95mm_HandSolder -> Capacitor_SMD:C_1206_3216Metric_Pad1.33x1.80mm_HandSolder; moved to B.Cu
- C56, C60: value 10uf -> 0.1uf; footprint Capacitor_SMD:C_0603_1608Metric_Pad1.08x0.95mm_HandSolder -> Capacitor_SMD:C_1206_3216Metric_Pad1.33x1.80mm_HandSolder; moved to B.Cu
- C57: value 0.1uf -> 22uf; footprint Capacitor_SMD:C_0603_1608Metric_Pad1.08x0.95mm_HandSolder -> Capacitor_SMD:C_1206_3216Metric_Pad1.33x1.80mm_HandSolder; moved to B.Cu
- C59: footprint Capacitor_SMD:C_0603_1608Metric_Pad1.08x0.95mm_HandSolder -> Capacitor_SMD:C_1206_3216Metric_Pad1.33x1.80mm_HandSolder; moved to B.Cu
- C61: value 0.1uf -> 10uf; footprint Capacitor_SMD:C_0603_1608Metric_Pad1.08x0.95mm_HandSolder -> Capacitor_SMD:C_1206_3216Metric_Pad1.33x1.80mm_HandSolder
- C62: value 27nf -> 10uf; footprint Capacitor_SMD:C_0603_1608Metric_Pad1.08x0.95mm_HandSolder -> Capacitor_SMD:C_1206_3216Metric_Pad1.33x1.80mm_HandSolder
- C63: value 1uf -> 0.1uf; footprint Capacitor_SMD:C_0603_1608Metric_Pad1.08x0.95mm_HandSolder -> Capacitor_SMD:C_1206_3216Metric_Pad1.33x1.80mm_HandSolder
- D2: value SMBJ58A -> SMBJ18CA; footprint Diode_SMD:D_SMA-SMB_Universal_Handsoldering -> Diode_SMD:D_SMB_Handsoldering
- D3: value SMBJ26A -> LED; footprint Diode_SMD:D_SMA-SMB_Universal_Handsoldering -> LED_SMD:LED_0805_2012Metric_Pad1.15x1.40mm_HandSolder
- D4: value LED -> SMBJ18CA; footprint LED_SMD:LED_0805_2012Metric_Pad1.15x1.40mm_HandSolder -> Diode_SMD:D_SMB_Handsoldering
- D5: value LED -> BAS516,115; footprint LED_SMD:LED_0805_2012Metric_Pad1.15x1.40mm_HandSolder -> Diode_SMD:D_SOD-523
- D6: value SK34SMA-3G -> D_Schottky; footprint Diode_SMD:D_SMA_Handsoldering -> Diode_SMD:D_SMB_Handsoldering
- D7, D8: value LED -> D_Schottky; footprint LED_SMD:LED_0805_2012Metric_Pad1.15x1.40mm_HandSolder -> Diode_SMD:D_SMB_Handsoldering
- D9: value SK34SMA-3G -> LED; footprint Diode_SMD:D_SMA_Handsoldering -> LED_SMD:LED_0805_2012Metric_Pad1.15x1.40mm_HandSolder
- FB1, FB2: moved to B.Cu
- J1: value PMOD_male_2row -> Conn_01x04_Socket; footprint ! Scott:PMOD_male_12pin -> Connector_JST:JST_EH_B4B-EH-A_1x04_P2.50mm_Vertical
- J8: value 1803426 -> 1758050; footprint ! Phoenix Contact:PHOENIX_1803426 -> ! Phoenix Contact:CONN_1758050
- J9: value 1758018 -> CU01SAH0S00; footprint ! Phoenix Contact:PHOENIX_1758018 -> ! Cvilux USA:CONN_CU01SAH0S00_CVI
- L6: value DRQ127-220-R -> 3.3uh; footprint ! Eaton:DRQ127 -> ! Bao Cheng Electronics:BCIHP10SC; moved to B.Cu
- R15: renamed from R10; value 51 -> 49.9
- R21: value 100K -> 10K
- R23: value 14.3K -> 78.7K; moved to B.Cu
- R24: value 10.5K -> 78.7K
- R26: renamed from R12; value 51 -> 49.9
- R28: renamed from R14; value 51 -> 49.9
- R3: renamed from R20; footprint Resistor_SMD:R_1206_3216Metric_Pad1.30x1.75mm_HandSolder -> Resistor_SMD:R_0603_1608Metric_Pad0.98x0.95mm_HandSolder
- R36: renamed from R16; value 51 -> 49.9
- R39: value 180K -> 10K; footprint Resistor_SMD:R_0603_1608Metric_Pad0.98x0.95mm_HandSolder -> Resistor_SMD:R_1206_3216Metric_Pad1.30x1.75mm_HandSolder; moved to B.Cu
- R42: value 2K -> 1K
- R44: value 75K -> 560; footprint Resistor_SMD:R_0603_1608Metric_Pad0.98x0.95mm_HandSolder -> Resistor_SMD:R_1206_3216Metric_Pad1.30x1.75mm_HandSolder
- R45: value 43.2K -> 68.4K; moved to B.Cu
- R46: value 180K -> 1.8K; footprint Resistor_SMD:R_0603_1608Metric_Pad0.98x0.95mm_HandSolder -> Resistor_SMD:R_1206_3216Metric_Pad1.30x1.75mm_HandSolder
- R47: footprint Resistor_SMD:R_0603_1608Metric_Pad0.98x0.95mm_HandSolder -> Resistor_SMD:R_1206_3216Metric_Pad1.30x1.75mm_HandSolder
- R48: value 10K -> 1.8K; footprint Resistor_SMD:R_0603_1608Metric_Pad0.98x0.95mm_HandSolder -> Resistor_SMD:R_1206_3216Metric_Pad1.30x1.75mm_HandSolder
- R5: renamed from R22; value 100K -> 107K
- U11: value LDL1117S50R_ -> MIC29302WU; footprint ! STMicroelectronics:SOT230P700X180-4N -> Package_TO_SOT_SMD:TO-263-5_TabPin3; moved to B.Cu
- U14: value LM5161PWP -> LDL1117S50R_; footprint Package_SO:Texas_HTSSOP-14-1EP_4.4x5mm_P0.65mm_EP3.4x5mm_Mask3.155x3.255mm_ThermalVias -> ! STMicroelectronics:SOT230P700X180-4N; moved to B.Cu
- moved TP5 179.8 mm to (139.9, -36.6)
- moved R48 171.3 mm to (134.9, -43.7)
- moved R44 171.1 mm to (134.9, -53.6)
- moved R46 170.0 mm to (134.9, -50.3)
- moved J16 159.0 mm to (180.0, 45.8), turned to 180 degrees
- moved H1 158.6 mm to (168.2, -84.4)
- moved TP4 157.5 mm to (125.8, -7.75)
- moved D9 149.0 mm to (107.8, -33.7), turned to 0 degrees
- moved H2 134.1 mm to (168.2, -76.5)
- moved TP8 129.9 mm to (139.9, -24.5)
- moved T5 128.5 mm to (164.3, 50.9), turned to -90 degrees
- moved R21 123.4 mm to (128.9, -50.3), turned to 0 degrees
- moved J1 121.8 mm to (60.0, 51.0), turned to -90 degrees
- moved TP7 118.7 mm to (139.9, -28.5)
- moved TP6 118.7 mm to (139.9, -32.6)
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- renumbered C12 to C18, C13 to C19, C29 to C2, C14 to C26, C15 to C27, C16 to C28, C17 to C29, C18 to C30, C19 to C31, C20 to C32, C21 to C33, C2 to C34, C22 to C35, C3 to C36, C4 to C37, C5 to C38, C6 to C39, C23 to C40, C7 to C41, C24 to C42, C25 to C43, C8 to C44, C9 to C45, C26 to C49, C27 to C51, C10 to C7, C11 to C9, J3 to J11, J4 to J12, J5 to J14, J6 to J15, J7 to J16, L1 to L2, L2 to L3, L3 to L4, L4 to L5, R9 to R14, R11 to R25, R13 to R27, R1 to R29, R2 to R30, R3 to R31, R4 to R32, R5 to R33, R15 to R34, R6 to R35, R7 to R37, R8 to R38, R17 to R40, R18 to R41, R19 to R43, U5 to U10, U6 to U12, U7 to U13, U2 to U5, U3 to U7, U4 to U8, U1 to U9
Connections:
- net Net-(J7-Ext) renamed /IRIG/IRIGGND
- C1 pad 1: GNDD -> +12V
- C1 pad 2: +3.3V -> GND
- C18 pad 1: +8VA -> /Distribution/Analog PWR
- C18 pad 2: GNDA -> /Distribution/Analog GND
- C19 pad 1: +8VA -> /Distribution/Analog PWR
- C19 pad 2: GNDA -> /Distribution/Analog GND
- C2 pad 1: Net-(D2-K) -> Net-(D2-A2)
- C27 pad 1: GNDA -> /Distribution/Analog GND
- C27 pad 2: Net-(J4-In) -> /Distribution/Buffer2/XFMRGND
- C28 pad 1: +8VA -> /Distribution/Analog PWR
- C28 pad 2: GNDA -> /Distribution/Analog GND
- C29 pad 1: +8VA -> /Distribution/Analog PWR
- C29 pad 2: GNDA -> /Distribution/Analog GND
- C31 pad 1: GNDA -> /Distribution/Analog GND
- C31 pad 2: Net-(J5-In) -> /Distribution/Buffer3/XFMRGND
- C32 pad 1: +8VA -> /Distribution/Analog PWR
- C32 pad 2: GNDA -> /Distribution/Analog GND
- C33 pad 1: +8VA -> /Distribution/Analog PWR
- C33 pad 2: GNDA -> /Distribution/Analog GND
- C36 pad 2: GNDA -> /Distribution/Analog GND
- C37 pad 2: GNDA -> /Distribution/Analog GND
- C38 pad 2: GNDA -> /Distribution/Analog GND
- C39 pad 2: GNDA -> /Distribution/Analog GND
- C40 pad 1: GNDA -> /Distribution/Analog GND
- C40 pad 2: Net-(J6-In) -> /Distribution/Buffer4/XFMRGND
- C41 pad 2: GNDA -> /Distribution/Analog GND
- C42 pad 1: +8VA -> /Distribution/Analog PWR
- C42 pad 2: GNDA -> /Distribution/Analog GND
- C43 pad 1: +8VA -> /Distribution/Analog PWR
- C43 pad 2: GNDA -> /Distribution/Analog GND
- C44 pad 1: +8VA -> /Distribution/Analog PWR
- C44 pad 2: GNDA -> /Distribution/Analog GND
- C45 pad 1: +8VA -> /Distribution/Analog PWR
- C45 pad 2: GNDA -> /Distribution/Analog GND
- C46 pad 1: +12V -> /IRIG/+11V IN
- C47 pad 1: +12V -> /Distribution/Analog PWR
- C47 pad 2: GND -> /Distribution/Analog GND
- C48 pad 1: Net-(C48-Pad1) -> +12V
- C48 pad 2: Net-(C48-Pad2) -> GND
- C50 pad 1: Net-(C48-Pad1) -> Net-(C50-Pad1)
- C51 pad 1: +5VA -> /IRIG/+5V IN
- C52 pad 1: Net-(U13-SS) -> +12V
- C53 pad 1: Net-(U13-FPWM) -> Net-(C53-Pad1)
- C54 pad 1: +6V -> Net-(U14-VIN)
- C54 pad 2: GND2 -> GND
- C55 pad 1: Net-(C55-Pad1) -> /IRIG/+5V IN
- C55 pad 2: Net-(U14-BST) -> GND
- C56 pad 1: +12V -> Net-(U15-VBST)
- C56 pad 2: GND -> Net-(U15-SW)
- C57 pad 1: +12V -> Net-(C53-Pad1)
- C58 pad 1: Net-(C58-Pad1) -> Net-(U11-EN)
- C58 pad 2: Net-(C58-Pad2) -> GND
- C59 pad 1: Net-(C58-Pad1) -> +12V
- C60 pad 1: Net-(C58-Pad1) -> +12V
- C61 pad 1: Net-(C58-Pad2) -> Net-(D8-K)
- C61 pad 2: Net-(U14-FB) -> /Distribution/Analog GND
- C62 pad 1: Net-(U14-SS) -> Net-(U16-EN)
- C62 pad 2: GND -> /Distribution/Analog GND
- C63 pad 1: Net-(U14-FPWM) -> Net-(D2-A2)
- C9 pad 1: GNDA -> /Distribution/Analog GND
- C9 pad 2: Net-(J3-In) -> /Distribution/Buffer1/XFMRGND
- D2 pad 1: Net-(D2-K) -> GND
- D2 pad 2: Net-(D2-A) -> Net-(D2-A2)
- D3 pad 1: GND -> Net-(D3-K)
- D3 pad 2: Net-(D2-A) -> Net-(D3-A)
- D4 pad 1: Net-(D4-K) -> GND
- D4 pad 2: +11VA -> Net-(D4-A2)
- D5 pad 2: +5VA -> Net-(D5-A)
- D6 pad 1: Net-(D6-K) -> /ocxo/+6V Analog
- D7 pad 1: Net-(D7-K) -> /ocxo/+6V Oven
- D7 pad 2: ISO_+8V -> Net-(D7-A)
- D8 pad 2: +12V -> Net-(D8-A)
- D9 pad 1: +6V -> Net-(D9-K)
- D9 pad 2: Net-(D9-A) -> /IRIG/+11V IN
- F1 pad 1: Net-(F1-Pad1) -> /power_connectors/+12Vin
- F1 pad 2: Net-(D2-K) -> Net-(D2-A2)
- FB1 pad 2: Net-(U9-EN) -> Net-(U11-EN)
- FB2 pad 1: Net-(U11-VIN) -> Net-(C53-Pad1)
- FB2 pad 2: Net-(U11-VIN) -> Net-(U14-VIN)
- FB3 pad 1: Net-(D6-K) -> Net-(D8-K)
- FB3 pad 2: Net-(U12-EN/UV) -> Net-(U16-EN)
- J1 pad 1: SPI_SDO -> GND
- J1 pad 2: ~{SPI_CS_OCXO} -> unconnected-(J1-Pin_2-Pad2)
- J1 pad 3: ~{SPI_CS_IRIG} -> /connectors/SDA
- J1 pad 4: unconnected-(J1-Pin_4-Pad4) -> /connectors/SCL
- J11 pad 1: Net-(J3-In) -> Net-(J11-In)
- J11 pad 2: Net-(J3-Ext) -> /Distribution/Buffer1/XFMRGND
- J12 pad 1: Net-(J4-In) -> Net-(J12-In)
- J12 pad 2: Net-(J4-Ext) -> /Distribution/Buffer2/XFMRGND
- J14 pad 1: Net-(J5-In) -> Net-(J14-In)
- J14 pad 2: Net-(J5-Ext) -> /Distribution/Buffer3/XFMRGND
- J15 pad 1: Net-(J6-In) -> Net-(J15-In)
- J15 pad 2: Net-(J6-Ext) -> /Distribution/Buffer4/XFMRGND
- J9 pad 1: Net-(F1-Pad1) -> Net-(U2-OUT)
- J9 pad 2: GND -> unconnected-(J9-Pad2)
- L5 pad 2: Net-(L4-Pad2) -> /Distribution/Buffer1/SINEIN
- L6 pad 1: Net-(C44-Pad1) -> Net-(U15-SW)
- L6 pad 2: ISO_GND8 -> Net-(C53-Pad1)
- Q1 pad 5: Net-(D2-K) -> Net-(D2-A2)
- R21 pad 1: Net-(D2-K) -> Net-(U6-DEMB)
- R21 pad 2: Net-(U8-EN/UVLO) -> GND
- R23 pad 1: Net-(U8-EN/UVLO) -> /IRIG/+11V IN
- R23 pad 2: GND -> Net-(U11-ADJ)
- R24 pad 1: Net-(U8-OVLO) -> /Distribution/Analog PWR
- R24 pad 2: GND -> Net-(U16-ADJ)
- R25 pad 1: /Distribution/Buffer2/SINEIN -> /Distribution/Buffer1/SINEIN
- R27 pad 1: /Distribution/Buffer3/SINEIN -> /Distribution/Buffer1/SINEIN
- R29 pad 2: +8VA -> /Distribution/Analog PWR
- R30 pad 1: ISO_10Mhz -> /Distribution/10Mhz
- R31 pad 1: GNDA -> /Distribution/Analog GND
- R33 pad 2: Net-(L4-Pad2) -> /Distribution/Buffer1/SINEIN
- R34 pad 1: /Distribution/Buffer4/SINEIN -> /Distribution/Buffer1/SINEIN
- R35 pad 2: +8VA -> /Distribution/Analog PWR
- R38 pad 1: GNDA -> /Distribution/Analog GND
- R39 pad 1: Net-(C44-Pad1) -> Net-(U11-ADJ)
- R39 pad 2: Net-(C48-Pad2) -> GND
- R42 pad 1: Net-(D8-K) -> Net-(U13-VOUT)
- R42 pad 2: GND -> Net-(C50-Pad1)
- R44 pad 1: +12V -> Net-(D10-K)
- R44 pad 2: Net-(U14-EN/UVLO) -> GND
- R45 pad 1: Net-(C58-Pad1) -> Net-(C53-Pad1)
- R45 pad 2: Net-(U14-FB) -> Net-(U15-VFB)
- R46 pad 1: Net-(C55-Pad1) -> Net-(D9-K)
- R46 pad 2: Net-(C58-Pad2) -> GND
- R47 pad 1: Net-(U14-EN/UVLO) -> Net-(U16-ADJ)
- R47 pad 2: GND -> /Distribution/Analog GND
- R48 pad 1: Net-(U14-FB) -> Net-(D11-K)
- R48 pad 2: GND -> /Distribution/Analog GND
- R5 pad 1: Net-(D2-K) -> Net-(D2-A2)
- R5 pad 2: Net-(U8-OVLO) -> Net-(U1-OVLO)
- T1 pad 3: GNDA -> /Distribution/Analog GND
- T1 pad 4: Net-(J3-In) -> /Distribution/Buffer1/XFMRGND
- T1 pad 6: Net-(J3-Ext) -> Net-(J11-In)
- T2 pad 3: GNDA -> /Distribution/Analog GND
- T2 pad 4: Net-(J4-In) -> /Distribution/Buffer2/XFMRGND
- T2 pad 6: Net-(J4-Ext) -> Net-(J12-In)
- T3 pad 3: GNDA -> /Distribution/Analog GND
- T3 pad 4: Net-(J5-In) -> /Distribution/Buffer3/XFMRGND
- T3 pad 6: Net-(J5-Ext) -> Net-(J14-In)
- T4 pad 3: GNDA -> /Distribution/Analog GND
- T4 pad 4: Net-(J6-In) -> /Distribution/Buffer4/XFMRGND
- T4 pad 6: Net-(J6-Ext) -> Net-(J15-In)
- TP2 pad 1: Net-(F1-Pad1) -> /power_connectors/+12Vin
- TP3 pad 1: +11VA -> Net-(D3-A)
- TP4 pad 1: Net-(U11-VIN) -> /power_connectors/+5Vin
- TP5 pad 1: +5VA -> /ocxo/GND Oven
- TP6 pad 1: Net-(D6-K) -> /IRIG/+5V IN
- TP7 pad 1: ISO_+8V -> Net-(C53-Pad1)
- TP8 pad 1: +6V -> /ocxo/GND Analog
- U10 pad 2: GNDA -> /Distribution/Analog GND
- U10 pad 5: +8VA -> /Distribution/Analog PWR
- U11 pad 1: GND -> Net-(U11-EN)
- U11 pad 2: +5VA -> Net-(U11-EN)
- U11 pad 3: Net-(U11-VIN) -> GND
- U11 pad 4: +5VA -> /IRIG/+11V IN
- U12 pad 3: Net-(U7-VOUT) -> Net-(C50-Pad1)
- U12 pad 5: +11VA -> /IRIG/+11V IN
- U13 pad 1: Net-(U7-VOUT) -> Net-(U13-VOUT)
- U13 pad 3: +5VA -> /IRIG/+5V IN
- U13 pad 4: SPI_SDO -> /IRIG/SPI_IRIG_MOSI
- U13 pad 5: SPI_SCLK -> /IRIG/SPI_IRIG_SCLK
- U13 pad 6: ~{SPI_CS_IRIG} -> /IRIG/~{SPI_IRIG_CS}
- U14 pad 2: GND -> /IRIG/+5V IN
- U14 pad 3: +12V -> Net-(U14-VIN)
- U14 pad 4: Net-(U14-EN/UVLO) -> /IRIG/+5V IN
- U5 pad 2: GNDA -> /Distribution/Analog GND
- U5 pad 5: +8VA -> /Distribution/Analog PWR
- U7 pad 2: GNDA -> /Distribution/Analog GND
- U7 pad 5: +8VA -> /Distribution/Analog PWR
- U8 pad 2: GNDA -> /Distribution/Analog GND
- U8 pad 5: +8VA -> /Distribution/Analog PWR
- U9 pad 2: GNDA -> /Distribution/Analog GND
- U9 pad 5: +8VA -> /Distribution/Analog PWR
Routing:
- net /Distribution/Analog GND: track 0.00 -> 331.7 mm, vias 0 -> 4
- net /Distribution/Analog PWR: track 0.00 -> 195.4 mm, vias 0 -> 4
- net /connectors/1PPS_FROM_GPS: track 0.00 -> 165.3 mm, vias 0 -> 1
- net /connectors/TX_FROM_GPS: track 0.00 -> 161.6 mm, vias 0 -> 1
- net /connectors/RX_TO_GPS: track 0.00 -> 160.2 mm, vias 0 -> 1
- net Net-(J17-Pin_18): track 0.00 -> 154.1 mm, vias 0 -> 1
- net /Distribution/Buffer1/SINEIN: track 46.5 -> 184.0 mm
- net Net-(J17-Pin_16): track 0.00 -> 126.0 mm, vias 0 -> 1
- net /ocxo/+6V Oven: track 0.00 -> 124.8 mm
- net GNDA: track 119.0 -> 0.00 mm
- net GND: track 58.9 -> 170.6 mm, vias 0 -> 1
- net /ocxo/+6V Analog: track 0.00 -> 93.6 mm
- net /connectors/SPI_MOSI: track 0.00 -> 81.4 mm, vias 0 -> 1
- net /ocxo/GND Analog: track 0.00 -> 79.4 mm
- net /connectors/SPI_SCLK: track 0.00 -> 75.8 mm, vias 0 -> 1
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- added copper zone on B.Cu, net /IRIG/IRIGGND
- added copper zone on F.Cu, net /IRIG/IRIGGND
Other:
- board size 140 x 127.5 mm -> 158 x 119 mm
- board text added: "FINTA Aux Board Version 1.0 2/15/26"
- board text added: "Heat"
