File: KiCAD/aux/power.kicad_sch (KiCad schematic)
At the start: 32 parts, among them J6 1803442, U10 LT3045xMSE, U11 LT1764AEQ_TRPBF, U9 LT3045xMSE

Commit message: Reworked, now with IRIG option board complete
Parts:
- removed C27, C28, C30, C33, C34, C35, C36, C37, C38, C40: 10uf, Capacitor_SMD:C_1206_3216Metric_Pad1.33x1.80mm_HandSolder, symbol Device:C
- removed C29, C39: 4.7uf, Capacitor_SMD:C_1206_3216Metric_Pad1.33x1.80mm_HandSolder, symbol Device:C
- removed J6: 1803442, ! Phoenix Contact:CONN_1803455, symbol ! Phoenix Contact:1803455
- removed NT1, NT2: NetTie_2, NetTie:NetTie-2_SMD_Pad0.5mm, symbol Device:NetTie_2
- removed NT3: NetTie_2, NetTie:NetTie-2_SMD_Pad2.0mm, symbol Device:NetTie_2
- removed R25: 2.5K, Resistor_SMD:R_0603_1608Metric_Pad0.98x0.95mm_HandSolder, symbol Device:R
- removed R26: 50K 0.05% 5ppm, Resistor_SMD:R_1206_3216Metric_Pad1.30x1.75mm_HandSolder, symbol Device:R
- removed R27: 3K, Resistor_SMD:R_1206_3216Metric_Pad1.30x1.75mm_HandSolder, symbol Device:R
- removed R28: 10.5K 0.05% 10ppm, Resistor_SMD:R_1206_3216Metric_Pad1.30x1.75mm_HandSolder, symbol Device:R
- removed R29: 3.32K 0.05% 10ppm, Resistor_SMD:R_1206_3216Metric_Pad1.30x1.75mm_HandSolder, symbol Device:R
- removed U10, U9: LT3045xMSE, Package_SO:MSOP-12-1EP_3x4.039mm_P0.65mm_EP1.651x2.845mm, symbol Regulator_Linear:LT3045xMSE
- removed U11: LT1764AEQ_TRPBF, ! Analog Devices:DDPAK-5_Q, symbol ! Analog Devices:LT1764AEQ_TRPBF
- added C10, C20, C24, C48, C53, C54, C55, C58, C59, C61, C62: 10uf, Capacitor_SMD:C_1206_3216Metric_Pad1.33x1.80mm_HandSolder, symbol Device:C
- added C11, C21, C25: 100uf polymer, Capacitor_THT:CP_Radial_D5.0mm_P2.00mm, symbol Device:C_Polarized
- added C12, C46, C47, C52, C57: 22uf, Capacitor_SMD:C_1206_3216Metric_Pad1.33x1.80mm_HandSolder, symbol Device:C
- added C13: 1uf, Capacitor_SMD:C_1206_3216Metric_Pad1.33x1.80mm_HandSolder, symbol Device:C
- added C14: 82pf, Capacitor_SMD:C_0402_1005Metric_Pad0.74x0.62mm_HandSolder, symbol Device:C
- added C15: 5.1pf, Capacitor_SMD:C_0402_1005Metric_Pad0.74x0.62mm_HandSolder, symbol Device:C
- added C16, C17: 39uf, Capacitor_SMD:C_1206_3216Metric_Pad1.33x1.80mm_HandSolder, symbol Device:C
- added C22: 33nf, Capacitor_SMD:C_0402_1005Metric_Pad0.74x0.62mm_HandSolder, symbol Device:C
- added C23: 150pf, Capacitor_SMD:C_0402_1005Metric_Pad0.74x0.62mm_HandSolder, symbol Device:C
- added C56, C60: 0.1uf, Capacitor_SMD:C_1206_3216Metric_Pad1.33x1.80mm_HandSolder, symbol Device:C
- added C8: 100nf, Capacitor_SMD:C_0603_1608Metric_Pad1.08x0.95mm_HandSolder, symbol Device:C
- added D10, D11, D9: LED, LED_SMD:LED_0805_2012Metric_Pad1.15x1.40mm_HandSolder, symbol Device:LED
- added D5: BAS516,115, Diode_SMD:D_SOD-523, symbol Device:D
- added D6, D7, D8: D_Schottky, Diode_SMD:D_SMB_Handsoldering, symbol Device:D_Schottky
- added L1: HP6-0090L, ! Coilcraft:HP6-0090L, symbol ! Coilcraft:HP6-0090L
- added L6: 3.3uh, ! Bao Cheng Electronics:BCIHP10SC, symbol ! Bao Cheng Electronics:BCIHP1040SC-3R3M
- added Q3, Q4: GSFD0650, Package_TO_SOT_SMD:TO-252-2, symbol Transistor_FET:Q_NMOS_GDS
- added R1: 1M, Resistor_SMD:R_0402_1005Metric_Pad0.72x0.64mm_HandSolder, symbol Device:R
- added R16: 2.26K, Resistor_SMD:R_0402_1005Metric_Pad0.72x0.64mm_HandSolder, symbol Device:R
- added R17: 25K, Resistor_SMD:R_0402_1005Metric_Pad0.72x0.64mm_HandSolder, symbol Device:R
- added R18: 210K, Resistor_SMD:R_0402_1005Metric_Pad0.72x0.64mm_HandSolder, symbol Device:R
- added R19: 50K, Resistor_SMD:R_0402_1005Metric_Pad0.72x0.64mm_HandSolder, symbol Device:R
- added R2: 15.4K, Resistor_SMD:R_0402_1005Metric_Pad0.72x0.64mm_HandSolder, symbol Device:R
- added R39, R47: 10K, Resistor_SMD:R_1206_3216Metric_Pad1.30x1.75mm_HandSolder, symbol Device:R
- added R44: 560, Resistor_SMD:R_1206_3216Metric_Pad1.30x1.75mm_HandSolder, symbol Device:R
- added R45: 68.4K, Resistor_SMD:R_0603_1608Metric_Pad0.98x0.95mm_HandSolder, symbol Device:R
- added R46, R48: 1.8K, Resistor_SMD:R_1206_3216Metric_Pad1.30x1.75mm_HandSolder, symbol Device:R
- added R49: 10K, Resistor_SMD:R_0603_1608Metric_Pad0.98x0.95mm_HandSolder, symbol Device:R
- added TP10, TP11, TP5, TP6, TP7, TP8, TP9: TestPoint_Probe, TestPoint:TestPoint_Pad_2.0x2.0mm, symbol Connector:TestPoint_Probe
- added U11, U16: MIC29302WU, Package_TO_SOT_SMD:TO-263-5_TabPin3, symbol Regulator_Linear:MIC29302WU
- added U14: LDL1117S50R_, ! STMicroelectronics:SOT230P700X180-4N, symbol ! STMicroelectronics:LDL1117S50R_
- added U15: TPS563201, Package_TO_SOT_SMD:SOT-23-6, symbol Regulator_Switching:TPS563201
- added U6: LM25116MHX_NOPB, ! Texas Instruments:SOP65P640X110-21N, symbol ! Texas Instruments:LM25116MHX_NOPB
- R20: value 80K 0.1% 50ppm -> 10mohm
- R21: value 2.5K -> 10K; footprint Resistor_SMD:R_0603_1608Metric_Pad0.98x0.95mm_HandSolder -> Resistor_SMD:R_1206_3216Metric_Pad1.30x1.75mm_HandSolder
- R22: value 66.5K -> 11.5K; footprint Resistor_SMD:R_0603_1608Metric_Pad0.98x0.95mm_HandSolder -> Resistor_SMD:R_0402_1005Metric_Pad0.72x0.64mm_HandSolder
- R23: value 3K -> 78.7K
- R24: value 31.6K -> 78.7K; footprint Resistor_SMD:R_0603_1608Metric_Pad0.98x0.95mm_HandSolder -> Resistor_SMD:R_1206_3216Metric_Pad1.30x1.75mm_HandSolder
Connections:
- net at R24.2: now also R47.1, U16.5 (ADJ)
- net at R20.1: now also Q4.3 (S), U6.12 (CS)
- net +11V IRIG: now reaches R23.1
- net +11V IRIG: now also C46.1, D9.2 (A), TP9.1, U11.4 (VOUT)
- net at FB1.2: now also C58.1, U11.1 (EN), U11.2 (VIN); no longer R22.1
- net at R22.2: now also C15.2, R18.1, R19.1, U6.8 (FB); no longer R21.1
- net +6V OCXO OSC: no longer names the net of FB3.1
- net +6V OCXO OSC: now also C10.1, C11.1, C61.1, D8.1 (K)
- net +6V OXCO Analog: no longer names the net of FB2.1
- net +6V OXCO Analog: now also C53.1, C57.1, L6.2, R45.1, TP7.1
- net +6V flt analog: no longer names the net of FB2.2
- net +6V flt analog: now also C54.1, U14.3 (VIN); no longer R24.1
- net +6V flt osc: no longer names the net of FB3.2
- net +6V flt osc: now also C62.1, U16.1 (EN), U16.2 (VIN)
- net +9V OXCO Analog renamed +12V
- net +12V: now also C12.1, C48.1, C52.1, C59.1, C60.1, R1.2, R2.2, U15.3 (VIN), U15.5 (EN), U6.1 (VIN)
- net GNDA renamed GND
- net GND: now also R22.1, C12.2, C13.2, C16.2, C17.2, C22.2, C23.2, C46.2, C48.2, C52.2, C53.2, C54.2, C55.2, C57.2, C58.2, C59.2, C60.2, R16.1, R17.1, R39.2, R44.2, R46.2, R49.2, U11.3 (GND), U14.1 (GND), U15.1 (GND), U6.13 (CSG), U6.14 (PGND), U6.21 (EP), U6.6 (AGND); no longer R23.2
- new net: D9.1 (K), R46.1
- new net: C13.1, D5.2 (A), Q3.2 (D), U6.16 (VCC)
- new net: C8.1, D5.1 (K), U6.18 (HB)
- new net: C8.2, L1.12, Q3.3 (S), Q4.2 (D), U6.20 (SW)
- new net: C56.2, L6.1, U15.2 (SW)
- new net: R45.2, R49.1, U15.4 (VFB)
- new net: C56.1, U15.6 (VBST)
- new net: Q3.1 (G), U6.19 (HO)
- new net: C22.1, U6.7 (SS)
- new net: R23.2, R39.1, U11.5 (ADJ)
- new net: D8.2 (A), L1.3
- new net: D10.1 (K), R44.1
- new net: C16.1, C17.1, L1.1, R19.2, U6.10 (VOUT), U6.17 (VCCX)
- new net: R21.1, U6.11 (DEMB)
- new net: Q4.1 (G), U6.15 (LO)
- new net: R16.2, R2.1, U6.2 (UVLO)
- new net: R17.2, U6.3 (RT/SYNC)
- new net: R1.1, U6.4 (EN)
- new net: C23.1, U6.5 (RAMP)
- new net: C14.1, C15.1, U6.9 (COMP)
- new net: D11.1 (K), R48.1
- new net: D6.2 (A), L1.6
- new net: C14.2, R18.2
- new net: L1.10, L1.2
- new net: D7.2 (A), L1.4, L1.5
- new net +11V Analog OCXO: C47.1, D11.2 (A), R24.1, TP10.1, U16.4 (VOUT)
- new net +5V IRIG: C55.1, D10.2 (A), TP6.1, U14.2 (VOUT), U14.4 (VOUT__1)
- new net +6V Analog OCXO: C24.1, C25.1, D6.1 (K)
- new net +6V OVEN OCXO: C20.1, C21.1, D7.1 (K)
- new net GND Analog  11V OCXO: C10.2, C11.2, C47.2, C61.2, C62.2, L1.11, R47.2, R48.2, TP11.1, U16.3 (GND)
- new net GND Analog 6V OCXO: C24.2, C25.2, L1.7, TP8.1
- new net GND OVEN OCXO: C20.2, C21.2, L1.8, L1.9, TP5.1
- no-connect marks 2 -> 0
Other:
- note removed: "OCXO Power"
