File: KiCAD/disciplined-ocxo/distribution.kicad_sch (KiCad schematic)
At the start: 22 parts, among them U9 AD8055ARTZ-R2

Commit message: Rework to real version 1.0, with separate GPS, OCXO, and IRIG boards
Parts:
- removed C34: 0.001uf C0G, Capacitor_SMD:C_1206_3216Metric_Pad1.33x1.80mm_HandSolder, symbol Device:C
- removed C36, C38: 390, Capacitor_SMD:C_1206_3216Metric_Pad1.33x1.80mm_HandSolder, symbol Device:C
- removed C37: 820, Capacitor_SMD:C_1206_3216Metric_Pad1.33x1.80mm_HandSolder, symbol Device:C
- removed C39: 0.1uf, Capacitor_SMD:C_1206_3216Metric_Pad1.33x1.80mm_HandSolder, symbol Device:C
- removed U9: AD8055ARTZ-R2, ! Analog Devices:SOT95P290X145-5N, symbol ! Analog Devices:AD8055ARTZ-R2
- added C43: 0.001uf C0G, Capacitor_SMD:C_1206_3216Metric_Pad1.33x1.80mm_HandSolder, symbol Device:C
- added C46, C48: 390pf C0G, Capacitor_SMD:C_1206_3216Metric_Pad1.33x1.80mm_HandSolder, symbol Device:C
- added C47: 820pf C0G, Capacitor_SMD:C_1206_3216Metric_Pad1.33x1.80mm_HandSolder, symbol Device:C
- added C49: 0.1uf C0G, Capacitor_SMD:C_1206_3216Metric_Pad1.33x1.80mm_HandSolder, symbol Device:C
- added U10: AD8055ARTZ-R2, ! Analog Devices:SOT95P290X145-5N, symbol ! Analog Devices:AD8055ARTZ-R2
- C44: value 0.1uf -> 0.1uf C0G
- C45: value 0.001uf -> 0.001uf C0G
- C50: renamed from C41; value 0.1uf -> 0.1uf C0G
- renumbered R29 to R24, R30 to R25, R31 to R26, R32 to R27, R33 to R28, R35 to R29, R37 to R30, R38 to R31
Connections:
- net Analog GND: now also C46.2, C47.2, C48.2, C49.2, U10.2 (V-)
- net Analog PWR: now also U10.5 (V+)
- net at L2.2, L3.1: now also C46.1
- net at L4.2, L5.1: now also C48.1
- net at R25.2: now also C43.1
- net at L3.2, L4.1: now also C47.1
- net at L2.1, R27.2: now also U10.1
- net at R27.1, R30.1: now also U10.4 (-)
- net at R24.1, R26.2: now also C43.2, U10.3 (+)
- net at R28.1: now also C49.1
Other:
- moved on the sheet: C45, C50, L2, L3, L4, L5, R24, R25, R26, R27, R28, R29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
