File: KiCAD/lownoise-LDO/lownoise-LDO.kicad_pcb (KiCad board)
At the start: 2 copper layers, 16.2 x 27 mm, 17 parts, among them J1 Conn_01x04_Pin, U1 LT3045xMSE

Commit message: LDO daughterboard 1.1
Parts:
- removed J1: Conn_01x04_Pin, Connector_PinHeader_2.00mm:PinHeader_1x04_P2.00mm_Horizontal
- removed the REF** at (115.7, 80.1)
- added FID1: Fiducial, Fiducial:Fiducial_1mm_Mask2mm, F.Cu at (114.6, 78.5)
- added FID2: Fiducial, Fiducial:Fiducial_1mm_Mask2mm, F.Cu at (127.8, 91.7)
- added FID3: Fiducial, Fiducial:Fiducial_1mm_Mask2mm, F.Cu at (114.6, 101.9)
- added J2: Conn_01x05_Pin, Connector_PinHeader_2.00mm:PinHeader_1x05_P2.00mm_Horizontal, B.Cu at (117.9, 100.3)
- added JP1: SolderJumper_2_Open, Jumper:SolderJumper-2_P1.3mm_Open_TrianglePad1.0x1.5mm, F.Cu at (123.2, 87.9)
- added REF**: KiCad-Logo2_5mm_SilkScreen, Symbol:KiCad-Logo2_5mm_SilkScreen, B.Cu at (121.4, 94.2)
- added REF**: ESD-Logo_6.6x6mm_SilkScreen, Symbol:ESD-Logo_6.6x6mm_SilkScreen, B.Cu at (116.8, 80.5)
Routing:
- net /GND: track 63.2 -> 50.2 mm
- net /SET: track 0.00 -> 12.9 mm
- net Net-(JP1-B): track 4.13 -> 7.95 mm
- net /+OUT: track 65.5 -> 64.6 mm
Other:
- board text added: "+IN"
- board text added: "+OUT"
- board text added: "GND"
- board text added: "LT3045 LDO Ver 1.1 5/14/26"
- board text added: "PG"
- board text added: "SET"
- board text removed: "CERN-OHL-S v2"
- board text removed: "LT3045 LDO"
- board text removed: "Ver 1.0 2/14/26"
