File: KiCAD/lownoise-LDO/lownoise-LDO.kicad_sch (KiCad schematic)
At the start: 16 parts, among them J1 Conn_01x04_Pin, U1 LT3045xMSE

Commit message: LDO daughterboard 1.1
Parts:
- removed J1: Conn_01x04_Pin, Connector_PinHeader_2.00mm:PinHeader_1x04_P2.00mm_Horizontal, symbol Connector:Conn_01x04_Pin
- added FID1, FID2, FID3: Fiducial, Fiducial:Fiducial_1mm_Mask2mm, symbol Mechanical:Fiducial
- added J2: Conn_01x05_Pin, Connector_PinHeader_2.00mm:PinHeader_1x05_P2.00mm_Horizontal, symbol Connector:Conn_01x05_Pin
- added JP1: SolderJumper_2_Open, Jumper:SolderJumper-2_P1.3mm_Open_TrianglePad1.0x1.5mm, symbol Jumper:SolderJumper_2_Open
Connections:
- net +IN: now also J2.1 (Pin_1)
- net +OUT: now also J2.3 (Pin_3)
- net GND: now also J2.2 (Pin_2)
- net PG: now also J2.4 (Pin_4)
- net at C4.1, R7.1, U1.8 (SET): now also JP1.2 (B)
- new net SET: J2.5 (Pin_5), JP1.1 (A)
